Commit message: update vehicle_param

File: logiee_vehicle_description/urdf/vehicle.xacro (robot description, xacro)
@@ -1,14 +1,91 @@
 <?xml version="1.0"?>
-<robot xmlns:xacro="http://ros.org/wiki/xacro">
-  <!-- load parameter -->
-  <xacro:property name="vehicle_info" value="${xacro.load_yaml('$(find logiee_vehicle_description)/config/vehicle_info.param.yaml')}"/>
+<robot xmlns:xacro="http://ros.org/wiki/xacro" name="logiee_vehicle">
+  <xacro:property name="vehicle_info" value="${load_yaml('$(find logiee_vehicle_description)/config/vehicle_info.param.yaml')}"/>
+  <xacro:property name="wheel_radius" value="${vehicle_info['/**']['ros__parameters']['wheel_radius']}"/>
+  <xacro:property name="wheel_width" value="${vehicle_info['/**']['ros__parameters']['wheel_width']}"/>
+  <xacro:property name="front_overhang" value="${vehicle_info['/**']['ros__parameters']['front_overhang']}"/>
+  <xacro:property name="rear_overhang" value="${vehicle_info['/**']['ros__parameters']['rear_overhang']}"/>
+  <xacro:property name="vehicle_width" value="0.5"/>
+  <xacro:property name="vehicle_length" value="0.6"/>
+  <xacro:property name="vehicle_height" value="${vehicle_info['/**']['ros__parameters']['vehicle_height']}"/>
+  <xacro:property name="caster_wheel_radius" value="0.08"/>
+  <!-- coordinate (x, y, 0) -->
+  <link name="base_footprint"/>
+  <joint name="virtual_footprint_joint" type="fixed">
+	<parent link="base_footprint"/>
+	<child link="base_link"/>
+	<origin xyz="0 0 ${wheel_radius}" rpy="0 0 0"/>
+  </joint>
+  <!-- the center of wheels (for control/planning) -->
+  <link name="base_link"/>
   <!-- vehicle body -->
-  <link name="base_link">
-    <visual>
-      <origin xyz="${vehicle_info['/**']['ros__parameters']['wheel_base']/2.0} 0 0" rpy="${pi/2.0} 0 ${pi}"/>
-      <geometry>
-        <mesh filename="package://sample_vehicle_description/mesh/logieeSSv1.dae" scale="1 1 1"/>
-      </geometry>
-    </visual>
+  <joint name="vehicle_body_joint" type="fixed">
+	<parent link="base_link"/>
+	<child link="vehicle_body"/>
+	<origin xyz="${vehicle_length/2 - rear_overhang} 0 ${wheel_radius}" rpy="0 0 0"/>
+  </joint>
+  <link name="vehicle_body">
+	<visual>
+	  <origin xyz="0 0 0" rpy="0 0 0"/>
+	  <geometry>
+		<box size="${vehicle_length} ${vehicle_width} ${vehicle_height}"/>
+	  </geometry>
+	  <material name="gray">
+		<color rgba="1.0 1.0 1.0 0.8"/>
+	  </material>
+	</visual>
+  </link>
+  <!-- two wheels -->
+  <!-- left wheel -->
+  <joint name="left_wheel_joint" type="fixed">
+	<origin xyz="0 -${vehicle_width/2.0} 0" rpy="0 0 0"/>
+	<parent link="base_link"/>
+	<child link="left_wheel_link"/>
+  </joint>
+  <link name="left_wheel_link">
+	<visual>
+	  <origin xyz="0 0 0 " rpy="-${pi/2} 0 0"/>
+	  <geometry>
+		<cylinder radius="${wheel_radius}" length="${wheel_width}"/>
+	  </geometry>
+	  <material name="red">
+		<color rgba="1.0 0.0 0.0 0.8"/>
+	  </material>
+	</visual>
+  </link>
+  <!-- right wheel -->
+  <joint name="right_wheel_joint" type="fixed">
+	<!-- if axis tag is not specified for continuous, the joint/link flickers -->
+	<origin xyz="0 ${vehicle_width/2.0} 0" rpy="0 0 0"/>
+	<parent link="base_link"/>
+	<child link="right_wheel_link"/>
+  </joint>
+  <link name="right_wheel_link">
+	<visual>
+	  <origin xyz="0 0 0 " rpy="-${pi/2} 0 0"/>
+	  <geometry>
+		<cylinder radius="${wheel_radius}" length="${wheel_width}"/>
+	  </geometry>
+	  <material name="red">
+		<color rgba="1.0 0.0 0.0 0.8"/>
+	  </material>
+	</visual>
+  </link>
+  <!-- front caster -->
+  <joint name="caster_joint" type="fixed">
+	<parent link="base_footprint"/>
+	<child link="caster_wheel"/>
+	<origin xyz="${front_overhang * 0.9} 0 ${caster_wheel_radius}" rpy="0 0 0"/>
+  </joint>
+  <link name="caster_wheel">
+	<visual>
+	  <origin xyz="0 0 0" rpy="${pi/2} 0 0"/>
+	  <geometry>
+		<cylinder radius="${caster_wheel_radius}" length="${wheel_width}"/>
+	  </geometry>
+	  <material name="white">
+		<color rgba="1.0 1.0 1.0 0.8"/>
+	  </material>
+	</visual>
   </link>
 </robot>
